File: plusd.sch (KiCad schematic (older format))
At the start: 52 parts, among them J1 Conn_02x17_Odd_Even, J2 ZX_Spectrum_Connector_GENERIC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, J3 Conn_02x13_Odd_Even, J4 Conn_01x03, SW1 SW_DPST_x2, SW2 SW_DIP_x02, U1 74LS06, U10 74LS27, U12 L7805, U2 AT28C256, U3 WD1772, U4 74LS00, U5 74LS126, U6 74LS175, U7 62256, U8 PAL20L8, U9 74LS374, Y1 8.000Mhz

Commit message: ahora con joystick
Parts:
- removed J3: Conn_02x13_Odd_Even, Connector_PinHeader_2.54mm:PinHeader_2x13_P2.54mm_Vertical, symbol Connector_Generic:Conn_02x13_Odd_Even
- removed U7: 62256, Package_DIP:DIP-28_W15.24mm_LongPads, symbol ALEA:62256
- added C18: 100n, Capacitors_THT:C_Disc_D5.0mm_W2.5mm_P5.00mm, symbol Device:C
- added D1: LED, LEDs:LED_D5.0mm, symbol Device:LED
- added J5: DB25_Female_MountingHoles, Connector_Dsub:DSUB-25_Female_Horizontal_P2.77x2.84mm_EdgePinOffset4.94mm_Housed_MountingHolesOffset7.48mm, symbol Connector:DB25_Female_MountingHoles
- added J6: Conn_02x13_Odd_Even, Connector_PinHeader_2.54mm:PinHeader_2x13_P2.54mm_Vertical, symbol Connector_Generic:Conn_02x13_Odd_Even
- added JP1: Jumper, Connector_PinHeader_2.54mm:PinHeader_1x02_P2.54mm_Vertical, symbol Device:Jumper
- added JP2: Conn_01x03, Connector_PinHeader_2.54mm:PinHeader_1x03_P2.54mm_Vertical, symbol Connector_Generic:Conn_01x03
- added JP4, JP5: Jumper_NC_Dual, Jumper:SolderJumper-3_P1.3mm_Bridged12_RoundedPad1.0x1.5mm, symbol Device:Jumper_NC_Dual
- added J_KEMPSTON_ATARI1: DB9_Male, Connector_Dsub:DSUB-9_Male_Horizontal_P2.77x2.84mm_EdgePinOffset4.94mm_Housed_MountingHolesOffset7.48mm, symbol plusd-rescue:DB9_Male-Connector_Specialized-All-Spectrums-rescue
- added MK3: Mounting_Hole, MountingHole:MountingHole_3mm, symbol Mechanical:Mounting_Hole
- added R2: 2K2, Resistors_THT:R_Axial_DIN0207_L6.3mm_D2.5mm_P7.62mm_Horizontal, symbol Device:R
- added SW3: SW_DPST_x2, Buttons_Switches_THT:SW_TH_Tactile_Omron_B3F-10xx, symbol Switch:SW_DPST_x2
- added U12: GAL22V10, Housings_DIP:DIP-24_W7.62mm_LongPads, symbol ALEA:GAL22V10
- added U6: 6264, Housings_DIP:DIP-28_W15.24mm_LongPads, symbol ALEA:6264
- C1: renamed from C4; footprint Capacitor_THT:C_Disc_D5.0mm_W2.5mm_P2.50mm -> Capacitors_THT:C_Disc_D5.0mm_W2.5mm_P5.00mm
- C10: renamed from C12; footprint Capacitor_THT:C_Disc_D5.0mm_W2.5mm_P2.50mm -> Capacitors_THT:C_Disc_D5.0mm_W2.5mm_P5.00mm
- C11: renamed from C13; footprint Capacitor_THT:C_Disc_D5.0mm_W2.5mm_P2.50mm -> Capacitors_THT:C_Disc_D5.0mm_W2.5mm_P5.00mm
- C12: renamed from C14; footprint Capacitor_THT:C_Disc_D5.0mm_W2.5mm_P2.50mm -> Capacitors_THT:C_Disc_D5.0mm_W2.5mm_P5.00mm
- C13: renamed from C15; footprint Capacitor_THT:C_Disc_D5.0mm_W2.5mm_P2.50mm -> Capacitors_THT:C_Disc_D5.0mm_W2.5mm_P5.00mm
- C14: renamed from C16; footprint Capacitor_THT:C_Disc_D5.0mm_W2.5mm_P2.50mm -> Capacitors_THT:C_Disc_D5.0mm_W2.5mm_P5.00mm
- C15: renamed from C2; footprint Capacitor_THT:C_Disc_D5.0mm_W2.5mm_P2.50mm -> Capacitors_THT:C_Disc_D5.0mm_W2.5mm_P2.50mm
- C16: renamed from C17; footprint Capacitor_THT:C_Disc_D5.0mm_W2.5mm_P2.50mm -> Capacitors_THT:C_Disc_D5.0mm_W2.5mm_P5.00mm
- C17: renamed from C1; value 100u -> 100u/16 V; footprint Capacitor_THT:CP_Radial_D7.5mm_P2.50mm -> Capacitors_THT:CP_Radial_D7.5mm_P2.50mm
- C2: renamed from C5; footprint Capacitor_THT:C_Disc_D5.0mm_W2.5mm_P2.50mm -> Capacitors_THT:C_Disc_D5.0mm_W2.5mm_P2.50mm
- C3: renamed from C6; value 100u -> 100u/16 V; footprint Capacitor_THT:CP_Radial_D7.5mm_P2.50mm -> Capacitors_THT:CP_Radial_D7.5mm_P2.50mm
- C4: renamed from C3; footprint Capacitor_THT:C_Disc_D5.0mm_W2.5mm_P2.50mm -> Capacitors_THT:C_Disc_D5.0mm_W2.5mm_P5.00mm
- C5: renamed from C7; value 100u -> 100u/16 V; footprint Capacitor_THT:CP_Radial_D7.5mm_P2.50mm -> Capacitors_THT:CP_Radial_D7.5mm_P2.50mm
- C6: renamed from C8; footprint Capacitor_THT:C_Disc_D5.0mm_W2.5mm_P2.50mm -> Capacitors_THT:C_Disc_D5.0mm_W2.5mm_P5.00mm
- C7: renamed from C9; footprint Capacitor_THT:C_Disc_D5.0mm_W2.5mm_P2.50mm -> Capacitors_THT:C_Disc_D5.0mm_W2.5mm_P5.00mm
- C8: renamed from C10; footprint Capacitor_THT:C_Disc_D5.0mm_W2.5mm_P2.50mm -> Capacitors_THT:C_Disc_D5.0mm_W2.5mm_P5.00mm
- C9: renamed from C11; footprint Capacitor_THT:C_Disc_D5.0mm_W2.5mm_P2.50mm -> Capacitors_THT:C_Disc_D5.0mm_W2.5mm_P5.00mm
- D2: renamed from D1; footprint Diode_THT:D_DO-35_SOD27_P7.62mm_Horizontal -> Diodes_THT:D_DO-35_SOD27_P7.62mm_Horizontal
- D3, D4: footprint Diode_THT:D_DO-35_SOD27_P7.62mm_Horizontal -> Diodes_THT:D_DO-35_SOD27_P7.62mm_Horizontal
- D5: renamed from D2; footprint LED_THT:LED_D5.0mm -> LEDs:LED_D5.0mm
- R1: renamed from R8; footprint Resistor_THT:R_Axial_DIN0207_L6.3mm_D2.5mm_P7.62mm_Horizontal -> Resistors_THT:R_Axial_DIN0207_L6.3mm_D2.5mm_P7.62mm_Horizontal
- R10: renamed from R6; footprint Resistor_THT:R_Axial_DIN0207_L6.3mm_D2.5mm_P7.62mm_Horizontal -> Resistors_THT:R_Axial_DIN0207_L6.3mm_D2.5mm_P7.62mm_Horizontal
- R11: renamed from R9; footprint Resistor_THT:R_Axial_DIN0207_L6.3mm_D2.5mm_P7.62mm_Horizontal -> Resistors_THT:R_Axial_DIN0207_L6.3mm_D2.5mm_P7.62mm_Horizontal
- R12: renamed from R7; footprint Resistor_THT:R_Axial_DIN0207_L6.3mm_D2.5mm_P7.62mm_Horizontal -> Resistors_THT:R_Axial_DIN0207_L6.3mm_D2.5mm_P7.62mm_Horizontal
- R3: renamed from R10; footprint Resistor_THT:R_Axial_DIN0207_L6.3mm_D2.5mm_P7.62mm_Horizontal -> Resistors_THT:R_Axial_DIN0207_L6.3mm_D2.5mm_P7.62mm_Horizontal
- R4: renamed from R11; footprint Resistor_THT:R_Axial_DIN0207_L6.3mm_D2.5mm_P7.62mm_Horizontal -> Resistors_THT:R_Axial_DIN0207_L6.3mm_D2.5mm_P7.62mm_Horizontal
- R5: renamed from R1; footprint Resistor_THT:R_Axial_DIN0207_L6.3mm_D2.5mm_P7.62mm_Horizontal -> Resistors_THT:R_Axial_DIN0207_L6.3mm_D2.5mm_P7.62mm_Horizontal
- R6: renamed from R2; footprint Resistor_THT:R_Axial_DIN0207_L6.3mm_D2.5mm_P7.62mm_Horizontal -> Resistors_THT:R_Axial_DIN0207_L6.3mm_D2.5mm_P7.62mm_Horizontal
- R7: renamed from R5; footprint Resistor_THT:R_Axial_DIN0207_L6.3mm_D2.5mm_P7.62mm_Horizontal -> Resistors_THT:R_Axial_DIN0207_L6.3mm_D2.5mm_P7.62mm_Horizontal
- R8: renamed from R3; footprint Resistor_THT:R_Axial_DIN0207_L6.3mm_D2.5mm_P7.62mm_Horizontal -> Resistors_THT:R_Axial_DIN0207_L6.3mm_D2.5mm_P7.62mm_Horizontal
- R9: renamed from R4; footprint Resistor_THT:R_Axial_DIN0207_L6.3mm_D2.5mm_P7.62mm_Horizontal -> Resistors_THT:R_Axial_DIN0207_L6.3mm_D2.5mm_P7.62mm_Horizontal
- SW1: footprint Button_Switch_THT:SW_TH_Tactile_Omron_B3F-10xx -> Buttons_Switches_THT:SW_TH_Tactile_Omron_B3F-10xx
- U1: renamed from U10; footprint Package_DIP:DIP-14_W7.62mm_LongPads -> Housings_DIP:DIP-14_W7.62mm_LongPads; symbol Logic_74xx:74LS27 -> plusd-rescue:74LS27-Logic_74xx
- U10: renamed from U9; footprint Package_DIP:DIP-20_W7.62mm_LongPads -> Housings_DIP:DIP-20_W7.62mm_LongPads; symbol Logic_74xx:74LS374 -> plusd-rescue:74LS374-Logic_74xx
- U11: renamed from U5; footprint Package_DIP:DIP-14_W7.62mm_LongPads -> Housings_DIP:DIP-14_W7.62mm_LongPads; symbol Logic_74xx:74LS126 -> plusd-rescue:74LS126-Logic_74xx
- U2: renamed from U8; footprint Package_DIP:DIP-24_W7.62mm_LongPads -> Housings_DIP:DIP-24_W7.62mm_LongPads
- U3: renamed from U4; footprint Package_DIP:DIP-14_W7.62mm_LongPads -> Housings_DIP:DIP-14_W7.62mm_LongPads; symbol Logic_74xx:74LS00 -> plusd-rescue:74LS00-Logic_74xx
- U4: renamed from U12; footprint Package_TO_SOT_THT:TO-220-3_Vertical -> TO_SOT_Packages_THT:TO-220-3_Vertical
- U5: renamed from U2; footprint Package_DIP:DIP-28_W15.24mm_LongPads -> Housings_DIP:DIP-28_W15.24mm_LongPads; symbol ALEA:AT28C256 -> plusd-rescue:AT28C256-ALEA
- U7: renamed from U3; footprint Package_DIP:DIP-28_W15.24mm_LongPads -> Housings_DIP:DIP-28_W15.24mm_LongPads; symbol ALEA:WD1772 -> plusd-rescue:WD1772-ALEA
- U8: renamed from U6; footprint Package_DIP:DIP-16_W7.62mm_LongPads -> Housings_DIP:DIP-16_W7.62mm_LongPads; symbol Logic_74xx:74LS175 -> plusd-rescue:74LS175-Logic_74xx
- U9: renamed from U1; footprint Package_DIP:DIP-14_W7.62mm_LongPads -> Housings_DIP:DIP-14_W7.62mm_LongPads; symbol Logic_74xx:74LS06 -> plusd-rescue:74LS06-Logic_74xx
- renumbered J2 to J1, J1 to J4, J4 to JP3, MK2 to MK1, MK1 to MK2
Connections:
- net labels added: ALT_MOTOR_ON, DIR, HEAD, INDEX, J1-Up, J2-Down, J3-Left, J4-Right, J6-Fire, MOTOR_ON, STEP, TRACK_0, plus3_5V
- net labels removed: XXX
- wire segments 429 -> 544
- no-connect marks 31 -> 36
Other:
- note added: "DATA_READ"
- note added: "DATA_WRITE\n"
- note added: "DENSITY SEL\n"
- note added: "DS0\n"
- note added: "DS1\n"
- note added: "GATE_WRITE\n"
- note added: "MOTOR 0\n"
- note added: "MOTOR 1"
- note added: "N/C"
- note added: "N/C\n"
- note added: "READY / DISK CHANGE\n"
- note added: "WRITE PROT"
- moved on the sheet: C1, C10, C11, C12, C13, C14, C15, C16, C17, C2, C3, C4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

Commit message: ahora con joystick
Connections:
- wire segments 544 -> 543
Changed lines of the file:
@@
 	10450 4800 10750 4800
-Wire Wire Line
-	10750 4800 10750 2650
 Wire Wire Line
 	10750 1950 11100 1950
@@
 Text Label 10750 2650 0    50   ~ 0
 TRACK_0
-Wire Wire Line
-	10750 2650 10750 1950
 Text Notes 11650 2050 0    50   ~ 0
 DS0\n
@@
 Wire Wire Line
 	10050 650  10450 650
-Connection ~ 10750 2650
 Wire Wire Line
 	10750 2650 11100 2650
@@
 Wire Bus Line
 	5950 850  5950 5900
+Wire Wire Line
+	10750 1950 10750 4800
 $EndSCHEMATC

Commit message: add cable jumpers
Parts:
- added JP4: Conn_01x04_Male, Connector_PinHeader_2.54mm:PinHeader_1x04_P2.54mm_Vertical, symbol Connector:Conn_01x04_Male
- R12, R2: value 2K2 -> 680
- renumbered JP4 to JP6
Connections:
- wire segments 543 -> 553
- no-connect marks 36 -> 35
Other:
- note added: "DS0"
- note added: "DS2"
- note added: "DS3"
- note added: "MODO XT: 2-3 (Cable plano, disqueteras DS0, DS1)\nMODO AT.: 1-2, 3-4 (Cable con cruze, ambas disqueteras DS1)"
- note added: "MOTOR"
- note added: "MOTOR 0"
- note added: "READY / Disc Chan."
- note removed: "MOTOR 0\n"
- note removed: "N/C\n"
- note removed: "READY / DISK CHANGE\n"
- moved on the sheet: C1, C4, J4, JP5, JP6, R1, R3, R4, SW3A, U12, U1A, U1B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

Commit message: fix power to chips
Parts:
- C2: value 10n -> 100n; footprint Capacitors_THT:C_Disc_D5.0mm_W2.5mm_P2.50mm -> Capacitors_THT:C_Disc_D5.0mm_W2.5mm_P5.00mm
Connections:
- wire segments 553 -> 539
- no-connect marks 35 -> 43
Other:
- moved on the sheet: JP2, U11A, U11C, U11D

Commit message: add schematic and BOM
Parts:
- added JP7: Conn_02x02_Odd_Even, Connector_PinHeader_2.54mm:PinHeader_2x02_P2.54mm_Vertical, symbol Connector_Generic:Conn_02x02_Odd_Even
Connections:
- wire segments 539 -> 549
- no-connect marks 43 -> 44
Other:
- note added: "normal: 1 y 2, 3 y 4, - DS0 es DS0 y DS1 es DS1\ninvertido: 1 y 3, 2 y 4 - DS0 es DS1 DS1 es DS0"
Changed lines of the file:
@@
 NoConn ~ 12100 1550
 NoConn ~ 12100 1650
-Text Label 10650 3200 1    50   ~ 0
+Text Label 10650 3100 1    50   ~ 0
 DS0
 Text Label 11900 1950 0    50   ~ 0
@@
 	10850 5250 10150 5250
 Wire Wire Line
-	10650 1400 10650 4400
+	10650 1400 10650 3150
 Wire Wire Line
 	10150 4400 10650 4400
@@
 	8700 950  8700 900
 Wire Wire Line
-	10750 1950 10750 4800
-Wire Wire Line
 	8950 2650 12100 2650
 Wire Wire Line
@@
 Wire Wire Line
 	9800 5550 9850 5550
+$Comp
+L Connector_Generic:Conn_02x02_Odd_Even JP7
+U 1 1 5B5832CA
+P 10750 3500
+F 0 "JP7" V 10754 3580 50  0000 L CNN
+F 1 "Conn_02x02_Odd_Even" V 10845 3580 50  0000 L CNN
+F 2 "Connector_PinHeader_2.54mm:PinHeader_2x02_P2.54mm_Vertical" H 10750 3500 50  0001 C CNN
+F 3 "~" H 10750 3500 50  0001 C CNN
+	1    10750 3500
+	0    1    1    0
+$EndComp
+Wire Wire Line
+	10650 4000 10450 4000
+Wire Wire Line
+	10450 4000 10450 3250
+Wire Wire Line
+	10450 3250 10650 3250
+Wire Wire Line
+	10650 3250 10650 3300
+Wire Wire Line
+	10650 4000 10650 4400
+Wire Wire Line
+	10650 3900 10650 3800
+Wire Wire Line
+	10650 3150 10350 3150
+Wire Wire Line
+	10350 3150 10350 3900
+Wire Wire Line
+	10350 3900 10650 3900
+Wire Wire Line
+	10750 1950 10750 3300
+Wire Wire Line
+	10750 3800 10750 4800
+Text Notes 10900 3850 0    50   ~ 0
+normal:   1 y 2, 3 y 4, - DS0 es DS0  y DS1 es DS1\ninvertido: 1 y 3, 2 y 4  - DS0 es DS1  DS1 es DS0
+NoConn ~ 11700 9550
 Wire Bus Line
 	850  2350 850  4550
@@
 	13600 550  13600 2400
 Wire Bus Line
-	8050 5900 8050 7400
-Wire Bus Line
 	15800 550  15800 2600
 Wire Bus Line
+	8050 5900 8050 7400
+Wire Bus Line
 	3500 4550 3500 6200
 Wire Bus Line
 	850  4550 850  6500
 Wire Bus Line
-	3500 550  3500 4550
-Wire Bus Line
 	5950 550  5950 5900
+Wire Bus Line
+	3500 550  3500 4550
 $EndSCHEMATC

Commit message: a
Parts:
- removed JP1: Jumper, Connector_PinHeader_2.54mm:PinHeader_1x02_P2.54mm_Vertical, symbol Device:Jumper
- C13: renamed from C15; footprint Capacitors_THT:C_Disc_D5.0mm_W2.5mm_P2.50mm -> Capacitor_THT:C_Disc_D5.0mm_W2.5mm_P5.00mm
- MK1: symbol Mechanical:Mounting_Hole_PAD -> plusd-rescue:Mounting_Hole_PAD-Mechanical
- MK2, MK3: symbol Mechanical:Mounting_Hole -> plusd-rescue:Mounting_Hole-Mechanical
- SW3: renamed from SW2; value SW_DIP_x02 -> SW_DIP_x03; footprint Button_Switch_THT:SW_DIP_SPSTx02_Slide_9.78x7.26mm_W7.62mm_P2.54mm -> Button_Switch_THT:SW_DIP_SPSTx03_Slide_6.7x9.18mm_W7.62mm_P2.54mm_LowProfile; symbol Switch:SW_DIP_x02 -> Switch:SW_DIP_x03
- renumbered C2 to C1, C13 to C10, C14 to C11, C16 to C12, C17 to C14, C1 to C15, C4 to C16, C3 to C17, C5 to C18, C6 to C2, C18 to C3, C7 to C4, C8 to C5, C9 to C6, C10 to C7, C11 to C8, C12 to C9, D4 to D2, D2 to D4, U7 to IC1, U1 to IC10, U12 to IC11, U4 to IC12, U5 to IC2, U6 to IC3, U2 to IC4, U9 to IC5, U11 to IC6, U10 to IC7, U8 to IC8, U3 to IC9, J4 to J2, J6 to J3, J_KEMPSTON_ATARI1 to J4, JP2 to JP1, JP3 to JP2, JP7 to JP5, JP5 to JP7, R5 to R1, R12 to R10, R3 to R11, R4 to R12, R6 to R2, R8 to R3, R9 to R4, R11 to R5, R2 to R6, R10 to R8, R1 to R9, SW3 to SW2
Connections:
- net labels added: JOY_EN
Other:
- moved on the sheet: R11, R12
