File: Rev_03/plusd.sch (KiCad schematic (older format))
At the start: 63 parts, among them J1 ZX_Spectrum_Connector_GENERIC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, J4 Conn_02x17_Odd_Even, J6 Conn_02x13_Odd_Even, SW1 SW_DPST_x2, SW2 SW_DIP_x02, SW3 SW_DPST_x2, U1 74LS27, U10 74LS374, U11 74LS126, U12 GAL22V10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

Commit message: aestetical changes
Connections:
- wire segments 498 -> 503
- no-connect marks 38 -> 33
Changed lines of the file:
@@
 EESchema Schematic File Version 4
+LIBS:plusd-cache
 EELAYER 26 0
 EELAYER END
@@
 Entry Wire Line
 	3500 5700 3600 5600
-Connection ~ 3500 4550
 Wire Wire Line
 	3600 6000 4650 6000
@@
 Text Label 1300 6400 0    50   ~ 0
 A2
-Wire Bus Line
-	850  4550 3500 4550
 $Comp
 L power:+5V #PWR05
@@
 Connection ~ 6450 10750
 Connection ~ 6450 11050
-Connection ~ 850  4550
 $Comp
 L plusd-rescue:74LS374-Logic_74xx U10
@@
 Entry Wire Line
 	5950 6300 6050 6400
-NoConn ~ 12900 6350
-NoConn ~ 12900 6250
-NoConn ~ 12900 6150
-NoConn ~ 12900 6050
 Wire Wire Line
 	12900 7150 13050 7150
@@
 Wire Wire Line
 	9800 5550 9850 5550
-NoConn ~ 12900 7250
 Wire Wire Line
 	8750 6050 12400 6050
@@
 Wire Wire Line
 	10750 1950 10750 4800
+Wire Wire Line
+	10650 1850 10650 4400
+Wire Wire Line
+	12900 6050 12900 6150
+Wire Wire Line
+	12900 6150 12900 6250
+Connection ~ 12900 6150
+Wire Wire Line
+	12900 6250 12900 6350
+Connection ~ 12900 6250
+Wire Wire Line
+	12900 6350 12900 6450
+Connection ~ 12900 6350
+Connection ~ 12900 6450
+Wire Wire Line
+	12900 7150 12900 7250
 Wire Bus Line
-	850  2350 850  4550
+	3500 550  850  550
 Wire Bus Line
 	13600 550  13600 2400
@@
 	8050 5900 8050 7400
 Wire Bus Line
-	3500 4550 3500 6200
-Wire Bus Line
-	850  4550 850  6500
-Wire Bus Line
 	5950 550  5950 5900
+Connection ~ 3500 550
 Wire Bus Line
-	3500 550  3500 4550
-Wire Wire Line
-	10650 1850 10650 4400
+	850  550  850  6500
+Wire Bus Line
+	3500 550  3500 6200
 $EndSCHEMATC
